File: HW3.X/Scott_Beck_PIC32/Scott_Beck_PIC32_Schematic.brd (EAGLE design)
At the start: 50 x 50 mm, 22 parts, among them J1 USB-MB-H

Commit message: First Complete Board
First Draft of Completed Board
Parts:
- C5, C6: device Scott_Beck_PIC32_Library:B45181B -> resistor:C0603
- LED1, LED2: device led:LED3MM -> led:SML0603
- moved R1 29.0 mm to (6.35, 3.81), turned to 270 degrees
- moved LED1 24.4 mm to (10.2, 3.81), turned to 90 degrees
- moved C3 10.2 mm to (21.6, 3.81)
- moved C4 6.35 mm to (14.0, 3.81), turned to 90 degrees
- moved C6 3.86 mm to (32.4, 19.5), turned to 270 degrees
- moved LED2 2.54 mm to (38.1, 47.0), turned to 270 degrees
- moved R3 1.63 mm to (12.4, 45.7), turned to 180 degrees
- moved C5 1.27 mm to (17.8, 3.81), turned to 90 degrees
- moved C1 0.43 mm to (34.3, 39.8)
- moved C2 0.31 mm to (17.8, 9.20)
- moved R4 0.25 mm to (12.4, 43.2)
Connections:
- net +3V3: now also C5.1; no longer C5.+
- net GND: now also C5.2, C6.2; no longer C5.-, C6.-
- net N$3: now also LED1.C; no longer LED1.K
- net N$5: now also C6.1; no longer C6.+
- net N$6: now also LED2.C; no longer LED2.K
Routing:
- net +3V3: track 0.00 -> 122.2 mm, vias 0 -> 3
- net A4/LED: track 0.00 -> 70.5 mm, vias 0 -> 2
- net B4/USER: track 0.00 -> 61.1 mm, vias 0 -> 1
- net +5V: track 0.00 -> 44.2 mm
- net D-: track 0.00 -> 30.2 mm
- net MCLR: track 0.00 -> 26.0 mm
- net D+: track 0.00 -> 25.5 mm
- net A1: track 0.00 -> 25.2 mm, vias 0 -> 2
- net A0: track 0.00 -> 25.2 mm, vias 0 -> 2
- net B9: track 0.00 -> 23.5 mm
- net B7: track 0.00 -> 23.5 mm
- net B8: track 0.00 -> 22.7 mm
- net USBID: track 0.00 -> 22.6 mm
- net N$8: track 0.00 -> 21.0 mm
- net N$7: track 0.00 -> 21.0 mm
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
Commit message: Semi-Finalized Board
Pre-Final Checks
Parts:
- moved J3 4.02 mm to (1.27, 16.5)
- moved U$6 3.24 mm to (1.27, 41.9)
- moved J2 1.91 mm to (48.8, 16.5)
- moved LED2 1.27 mm to (36.8, 47.0)
- moved J1 1.27 mm to (45.7, 6.35)
Connections:
- net N$7 renamed PGD
- net N$8 renamed PGC
Routing:
- net +3V3: track 122.2 -> 129.3 mm
- net B4/USER: track 61.1 -> 64.0 mm
- net A1: track 25.2 -> 22.6 mm
- net A0: track 25.2 -> 22.6 mm
- net PGD: track 21.0 -> 23.0 mm
- net PGC: track 21.0 -> 23.0 mm
- net A4/LED: track 70.5 -> 72.1 mm
- net B8: track 22.7 -> 24.3 mm
- net +5V: track 44.2 -> 45.7 mm
- net N$6: track 3.85 -> 2.58 mm
- net D+: track 25.5 -> 24.2 mm
- net D-: track 30.2 -> 28.9 mm
- net USBID: track 22.6 -> 23.7 mm
- net B7: track 23.5 -> 24.3 mm
- net B9: track 23.5 -> 24.3 mm
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Other:
- board text added: "3V3"
- board text added: "5V"
- board text added: "A0"
- board text added: "A1"
- board text added: "A4/LED"
- board text added: "April 7, 2017"
- board text added: "B13"
- board text added: "B14"
- board text added: "B15"
- board text added: "B2"
- board text added: "B3"
- board text added: "B4/USER"
- board text added: "B7"
- board text added: "B8"
- board text added: "B9"
- board text added: "GND"
- board text added: "Scott Beck"

Commit message: GERBER Files
Finalized Board and Made GERBER Files
Parts:
- moved LED1 0.64 mm to (9.54, 3.70), turned to 270 degrees
- moved C3 0.64 mm to (21.0, 3.81)
- moved C5 0.64 mm to (17.1, 3.81)
- moved C4 0.63 mm to (13.3, 3.81)
- moved R1 0.60 mm to (5.75, 3.84), turned to 90 degrees
Routing:
- net +3V3: track 129.3 -> 138.7 mm
- net +5V: track 45.7 -> 46.3 mm
